File: kuc.kicad_sch (KiCad schematic)
At the start: 57 parts, among them J2 KUC

Commit message: added schematic details
Other:
- company: (none) -> W3AXL
- title: (none) -> Kenwood Universal Connector
Changed lines of the file:
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@@
 (kicad_sch (version 20211123) (generator eeschema)
-  (paper "A4")
+  (paper "USLetter")
+  (title_block
+    (title "Kenwood Universal Connector")
+    (date "2023-05-28")
+    (rev "A")
+    (company "W3AXL")
+  )
   (junction (at 139.7 92.71) (diameter 0) (color 0 0 0 0)
   )
